File: PanelInterconnect.kicad_pcb (KiCad board)
At the start: 2 copper layers, 1144.8 x 86.1 mm, 10 parts, among them J1 Conn_01x10, J3 Conn_01x30

Commit message: Panelizing interconnects
Parts:
- removed the J1 at (5.60, 408.4)
- removed the J3 at (1173.2, 409.9)
- removed the SC1 at (134.2, 409.2)
- removed the SC2 at (264.2, 409.2)
- removed the SC3 at (394.2, 409.2)
- removed the SC4 at (524.2, 409.2)
- removed the SC5 at (654.2, 409.2)
- removed the SC6 at (784.2, 409.2)
- removed the SC7 at (914.2, 409.2)
- removed the SC8 at (1044.2, 409.2)
- added J1: Conn_01x10, _PanelInterconnct:kyocera_fpc_01x10, F.Cu at (-4.90, 558.2)
- added J1: Conn_01x10, _PanelInterconnct:kyocera_fpc_01x10, F.Cu at (-4.90, 428.2)
- added J1: Conn_01x10, _PanelInterconnct:kyocera_fpc_01x10, F.Cu at (25.1, 493.2)
- added J1: Conn_01x10, _PanelInterconnct:kyocera_fpc_01x10, F.Cu at (25.1, 363.2)
- added J1: Conn_01x10, _PanelInterconnct:kyocera_fpc_01x10, F.Cu at (-6.40, 299.4)
- added J3: Conn_01x30, _PanelInterconnct:kyocera_fpc_01x30, F.Cu at (1162.8, 559.7)
- added J3: Conn_01x30, _PanelInterconnct:kyocera_fpc_01x30, F.Cu at (1192.8, 494.7)
- added J3: Conn_01x30, _PanelInterconnct:kyocera_fpc_01x30, F.Cu at (1192.8, 364.7)
- added J3: Conn_01x30, _PanelInterconnct:kyocera_fpc_01x30, F.Cu at (1161.2, 300.9)
- added J3: Conn_01x30, _PanelInterconnct:kyocera_fpc_01x30, F.Cu at (1162.8, 429.7)
- added SC1: Maxeon C60, _PanelInterconnct:maxeon_c60, F.Cu at (123.8, 559.0)
- added SC1: Maxeon C60, _PanelInterconnct:maxeon_c60, F.Cu at (123.8, 429.0)
- added SC1: Maxeon C60, _PanelInterconnct:maxeon_c60, F.Cu at (122.2, 300.2)
- added SC1: Maxeon C60, _PanelInterconnct:maxeon_c60, F.Cu at (153.8, 364.0)
- added SC1: Maxeon C60, _PanelInterconnct:maxeon_c60, F.Cu at (153.8, 494.0)
- added SC2: Maxeon C60, _PanelInterconnct:maxeon_c60, F.Cu at (253.8, 429.0)
- added SC2: Maxeon C60, _PanelInterconnct:maxeon_c60, F.Cu at (252.2, 300.2)
- added SC2: Maxeon C60, _PanelInterconnct:maxeon_c60, F.Cu at (253.8, 559.0)
- added SC2: Maxeon C60, _PanelInterconnct:maxeon_c60, F.Cu at (283.8, 494.0)
- added SC2: Maxeon C60, _PanelInterconnct:maxeon_c60, F.Cu at (283.8, 364.0)
- added SC3: Maxeon C60, _PanelInterconnct:maxeon_c60, F.Cu at (413.8, 494.0)
- added SC3: Maxeon C60, _PanelInterconnct:maxeon_c60, F.Cu at (383.8, 429.0)
- added SC3: Maxeon C60, _PanelInterconnct:maxeon_c60, F.Cu at (413.8, 364.0)
- added SC3: Maxeon C60, _PanelInterconnct:maxeon_c60, F.Cu at (383.8, 559.0)
- added SC3: Maxeon C60, _PanelInterconnct:maxeon_c60, F.Cu at (382.2, 300.2)
- added SC4: Maxeon C60, _PanelInterconnct:maxeon_c60, F.Cu at (543.8, 364.0)
- added SC4: Maxeon C60, _PanelInterconnct:maxeon_c60, F.Cu at (513.8, 559.0)
- added SC4: Maxeon C60, _PanelInterconnct:maxeon_c60, F.Cu at (512.2, 300.2)
- added SC4: Maxeon C60, _PanelInterconnct:maxeon_c60, F.Cu at (543.8, 494.0)
- added SC4: Maxeon C60, _PanelInterconnct:maxeon_c60, F.Cu at (513.8, 429.0)
- added SC5: Maxeon C60, _PanelInterconnct:maxeon_c60, F.Cu at (642.2, 300.2)
- added SC5: Maxeon C60, _PanelInterconnct:maxeon_c60, F.Cu at (673.8, 364.0)
- added SC5: Maxeon C60, _PanelInterconnct:maxeon_c60, F.Cu at (673.8, 494.0)
- added SC5: Maxeon C60, _PanelInterconnct:maxeon_c60, F.Cu at (643.8, 559.0)
- added SC5: Maxeon C60, _PanelInterconnct:maxeon_c60, F.Cu at (643.8, 429.0)
- added SC6: Maxeon C60, _PanelInterconnct:maxeon_c60, F.Cu at (772.2, 300.2)
- added SC6: Maxeon C60, _PanelInterconnct:maxeon_c60, F.Cu at (803.8, 364.0)
- added SC6: Maxeon C60, _PanelInterconnct:maxeon_c60, F.Cu at (773.8, 559.0)
- added SC6: Maxeon C60, _PanelInterconnct:maxeon_c60, F.Cu at (803.8, 494.0)
- added SC6: Maxeon C60, _PanelInterconnct:maxeon_c60, F.Cu at (773.8, 429.0)
- added SC7: Maxeon C60, _PanelInterconnct:maxeon_c60, F.Cu at (933.8, 494.0)
- added SC7: Maxeon C60, _PanelInterconnct:maxeon_c60, F.Cu at (903.8, 559.0)
- added SC7: Maxeon C60, _PanelInterconnct:maxeon_c60, F.Cu at (903.8, 429.0)
- added SC7: Maxeon C60, _PanelInterconnct:maxeon_c60, F.Cu at (933.8, 364.0)
- added SC7: Maxeon C60, _PanelInterconnct:maxeon_c60, F.Cu at (902.2, 300.2)
- added SC8: Maxeon C60, _PanelInterconnct:maxeon_c60, F.Cu at (1033.8, 429.0)
- added SC8: Maxeon C60, _PanelInterconnct:maxeon_c60, F.Cu at (1063.8, 364.0)
- added SC8: Maxeon C60, _PanelInterconnct:maxeon_c60, F.Cu at (1063.8, 494.0)
- added SC8: Maxeon C60, _PanelInterconnct:maxeon_c60, F.Cu at (1033.8, 559.0)
- added SC8: Maxeon C60, _PanelInterconnct:maxeon_c60, F.Cu at (1032.2, 300.2)
Routing:
- net Net-(J1-Pin_1): track 1157.1 -> 5785.6 mm, vias 10 -> 50
- net Net-(J1-Pin_10): track 41.0 -> 205.2 mm, vias 21 -> 105
- net Net-(J3-Pin_1): track 30.5 -> 152.7 mm
Other:
- board size 1144.8 x 86.1 mm -> 1200 x 375 mm
