File: PanelInterconnect.kicad_pcb (KiCad board)
At the start: 2 copper layers, 14 parts, among them J1 Conn_01x02, J2 Conn_01x04

Commit message: Pushing
Parts:
- removed J1: Conn_01x02, TerminalBlock:TerminalBlock_MaiXu_MX126-5.0-02P_1x02_P5.00mm
- added J3: Conn_01x30, _PanelInterconnct:FPC_30x01, F.Cu at (1363.0, 396.6)
- J2: value Conn_01x04 -> Conn_01x06; footprint TerminalBlock:TerminalBlock_MaiXu_MX126-5.0-04P_1x04_P5.00mm -> Connector_FFC-FPC:Jushuo_AFC07-S06FCA-00_1x6-1MP_P0.50_Horizontal
- moved J2 235.5 mm to (-212.1, 399.2)
Connections:
- J2 pad 1: Net-(J1-Pin_1) -> Net-(J2-Pin_1)
- J2 pad 2: Net-(J1-Pin_2) -> Net-(J2-Pin_1)
- J2 pad 3: Net-(J2-Pin_3) -> Net-(J2-Pin_1)
- SC1 pad 1: Net-(J2-Pin_3) -> Net-(J2-Pin_4)
- SC12 pad 2: Net-(J2-Pin_4) -> Net-(J3-Pin_1)
Routing:
- added copper zone on B.Cu, net Net-(SC10-+)
- added copper zone on B.Cu, net Net-(SC10--)
- added copper zone on B.Cu, net Net-(SC4--)
- added copper zone on B.Cu, net Net-(SC5--)
- added copper zone on B.Cu, net Net-(SC6--)
- added copper zone on B.Cu, net Net-(SC7--)
- added copper zone on B.Cu, net Net-(SC8--)
- removed copper zone on F.Cu, net Net-(SC1--)
Other:
- board outline added: 1523 x 86 mm

Commit message: Still working on it
Parts:
- removed J2: Conn_01x06, Connector_FFC-FPC:Jushuo_AFC07-S06FCA-00_1x6-1MP_P0.50_Horizontal
- removed SC10, SC11, SC12, SC9: Solar_Cell, _PanelInterconnct:maxeon_c60
- added J1: Conn_01x10, _PanelInterconnct:kyocera_fpc_01x10, F.Cu at (74.0, 398.2)
- J3: footprint _PanelInterconnct:FPC_30x01 -> _PanelInterconnct:kyocera_fpc_01x30
- moved SC2 273.5 mm to (293.5, 399.0)
- moved SC3 273.5 mm to (420.5, 399.0)
- moved SC4 273.5 mm to (547.5, 399.0)
- moved SC5 273.5 mm to (674.5, 399.0)
- moved SC6 273.5 mm to (801.5, 399.0)
- moved SC7 273.5 mm to (928.5, 399.0)
- moved SC8 273.5 mm to (1055.5, 399.0)
- moved SC1 272.5 mm to (165.5, 399.0)
- moved J3 218.9 mm to (1144.2, 399.7)
Connections:
- SC8 pad 2: Net-(SC8--) -> Net-(J3-Pin_1)
Routing:
- net Net-(J1-Pin_1): track 0.00 -> 1070.6 mm, vias 0 -> 5
- net Net-(J1-Pin_4): track 0.00 -> 60.0 mm, vias 0 -> 18
- net Net-(J3-Pin_1): track 0.00 -> 26.0 mm
- net (no net): vias 0 -> 2
- added copper zone on B.Cu, net Net-(J1-Pin_4)
- added copper zone on F.Cu, net Net-(J1-Pin_4)
- added copper zone on B.Cu, net Net-(J3-Pin_1)
- added copper zone on F.Cu, net Net-(J3-Pin_1)
- added copper zone on F.Cu, net Net-(SC1--)
- added copper zone on F.Cu, net Net-(SC2--)
- added copper zone on F.Cu, net Net-(SC3--)
- added copper zone on F.Cu, net Net-(SC4--)
- added copper zone on F.Cu, net Net-(SC5--)
- added copper zone on F.Cu, net Net-(SC6--)
- added copper zone on F.Cu, net Net-(SC7--)
- removed copper zone on B.Cu, net Net-(SC1--)
- removed copper zone on B.Cu, net Net-(SC10-+)
- removed copper zone on B.Cu, net Net-(SC10--)
- removed copper zone on B.Cu, net Net-(SC2--)
- removed copper zone on B.Cu, net Net-(SC3--)
- removed copper zone on B.Cu, net Net-(SC4--)
- removed copper zone on B.Cu, net Net-(SC5--)
- removed copper zone on B.Cu, net Net-(SC6--)
- removed copper zone on B.Cu, net Net-(SC7--)
- removed copper zone on B.Cu, net Net-(SC8--)
Other:
- board size 1523 x 86 mm -> 1047.3 x 86 mm
- board text added: "SC2"
- board text added: "Solar_Cell"

Commit message: Working on it still
Parts:
- SC1, SC2, SC3, SC4, SC5, SC6, SC7, SC8: value Solar_Cell -> Maxeon C60
- moved J3 20.5 mm to (1164.7, 399.7)
- moved SC8 20.0 mm to (1075.5, 399.0)
- moved SC7 17.0 mm to (945.5, 399.0)
- moved SC6 14.0 mm to (815.5, 399.0)
- moved SC5 11.0 mm to (685.5, 399.0)
- moved SC4 8.00 mm to (555.5, 399.0)
- moved SC3 5.00 mm to (425.5, 399.0)
- moved SC2 2.00 mm to (295.5, 399.0)
Routing:
- net Net-(J1-Pin_4): track 60.0 -> 80.5 mm
- net Net-(J1-Pin_1): track 1070.6 -> 1091.1 mm
Other:
- board size 1047.3 x 86 mm -> 1067.8 x 86 mm

Commit message: Cleaning up layout
Parts:
- moved J1 69.1 mm to (5.60, 408.4)
- moved SC1 32.9 mm to (134.2, 409.2), turned to -90 degrees
- moved SC2 32.9 mm to (264.2, 409.2), turned to -90 degrees
- moved SC3 32.9 mm to (394.2, 409.2), turned to -90 degrees
- moved SC4 32.9 mm to (524.2, 409.2), turned to -90 degrees
- moved SC5 32.9 mm to (654.2, 409.2), turned to -90 degrees
- moved SC6 32.9 mm to (784.2, 409.2), turned to -90 degrees
- moved SC7 32.9 mm to (914.2, 409.2), turned to -90 degrees
- moved SC8 32.9 mm to (1044.2, 409.2), turned to -90 degrees
- moved J3 13.4 mm to (1173.2, 409.9)
Connections:
- J1 pad 10: unconnected-(J1-Pin_10-Pad10) -> Net-(J1-Pin_10)
- J1 pad 4: Net-(J1-Pin_4) -> unconnected-(J1-Pin_4-Pad4)
- J1 pad 5: Net-(J1-Pin_4) -> Net-(J1-Pin_10)
- J1 pad 6: Net-(J1-Pin_4) -> Net-(J1-Pin_10)
- J1 pad 7: unconnected-(J1-Pin_7-Pad7) -> Net-(J1-Pin_10)
- J1 pad 8: unconnected-(J1-Pin_8-Pad8) -> Net-(J1-Pin_10)
- J1 pad 9: unconnected-(J1-Pin_9-Pad9) -> Net-(J1-Pin_10)
- J3 pad 15: Net-(J1-Pin_4) -> Net-(J1-Pin_10)
- J3 pad 16: Net-(J1-Pin_4) -> Net-(J1-Pin_10)
- J3 pad 17: Net-(J1-Pin_4) -> Net-(J1-Pin_10)
- J3 pad 18: Net-(J1-Pin_4) -> Net-(J1-Pin_10)
- J3 pad 19: Net-(J1-Pin_4) -> Net-(J1-Pin_10)
- J3 pad 20: Net-(J1-Pin_4) -> Net-(J1-Pin_10)
- J3 pad 21: Net-(J1-Pin_4) -> Net-(J1-Pin_10)
- J3 pad 22: Net-(J1-Pin_4) -> Net-(J1-Pin_10)
- J3 pad 23: Net-(J1-Pin_4) -> Net-(J1-Pin_10)
- J3 pad 24: Net-(J1-Pin_4) -> Net-(J1-Pin_10)
- J3 pad 25: Net-(J1-Pin_4) -> Net-(J1-Pin_10)
- J3 pad 26: Net-(J1-Pin_4) -> Net-(J1-Pin_10)
- J3 pad 27: Net-(J1-Pin_4) -> Net-(J1-Pin_10)
- SC1 pad 1: Net-(J1-Pin_4) -> Net-(SC1-+)
- SC1 pad 2: Net-(SC1--) -> Net-(J1-Pin_10)
- SC2 pad 1: Net-(SC1--) -> Net-(SC2-+)
- SC2 pad 2: Net-(SC2--) -> Net-(SC1-+)
- SC3 pad 1: Net-(SC2--) -> Net-(SC3-+)
- SC3 pad 2: Net-(SC3--) -> Net-(SC2-+)
- SC4 pad 1: Net-(SC3--) -> Net-(SC4-+)
- SC4 pad 2: Net-(SC4--) -> Net-(SC3-+)
- SC5 pad 1: Net-(SC4--) -> Net-(SC5-+)
- SC5 pad 2: Net-(SC5--) -> Net-(SC4-+)
- SC6 pad 1: Net-(SC5--) -> Net-(SC6-+)
- SC6 pad 2: Net-(SC6--) -> Net-(SC5-+)
- SC7 pad 1: Net-(SC6--) -> Net-(SC7-+)
- SC7 pad 2: Net-(SC7--) -> Net-(SC6-+)
- SC8 pad 1: Net-(SC7--) -> Net-(J3-Pin_1)
- SC8 pad 2: Net-(J3-Pin_1) -> Net-(SC7-+)
Routing:
- net Net-(J1-Pin_4): track 80.5 -> 0.00 mm, vias 18 -> 0
- net Net-(J1-Pin_1): track 1091.1 -> 1161.0 mm, vias 5 -> 8
- net Net-(J1-Pin_10): track 0.00 -> 41.0 mm, vias 0 -> 21
- net Net-(J3-Pin_1): track 26.0 -> 30.5 mm
- net (no net): vias 2 -> 0
- added copper zone on B.Cu, net Net-(J1-Pin_1)
- added copper zone on F.Cu, net Net-(J1-Pin_1)
- added copper zone on B.Cu, net Net-(J1-Pin_10)
- added copper zone on F.Cu, net Net-(J1-Pin_10)
- added copper zone on F.Cu, net Net-(SC1-+)
- added copper zone on F.Cu, net Net-(SC2-+)
- added copper zone on F.Cu, net Net-(SC3-+)
- added copper zone on F.Cu, net Net-(SC4-+)
- added copper zone on F.Cu, net Net-(SC5-+)
- added copper zone on F.Cu, net Net-(SC6-+)
- added copper zone on F.Cu, net Net-(SC7-+)
- removed copper zone on B.Cu, net Net-(J1-Pin_4)
- removed copper zone on F.Cu, net Net-(J1-Pin_4)
- removed copper zone on F.Cu, net Net-(SC1--)
- removed copper zone on F.Cu, net Net-(SC2--)
- removed copper zone on F.Cu, net Net-(SC3--)
- removed copper zone on F.Cu, net Net-(SC4--)
- removed copper zone on F.Cu, net Net-(SC5--)
- removed copper zone on F.Cu, net Net-(SC6--)
- removed copper zone on F.Cu, net Net-(SC7--)
Other:
- board size 1067.8 x 86 mm -> 1144.8 x 86 mm

Commit message: Adding finishing touches to PCB and adding fab outputs
Routing:
- net Net-(J1-Pin_1): track 1161.0 -> 1157.1 mm, vias 8 -> 10
Other:
- board size 1144.8 x 86 mm -> 1144.8 x 86.1 mm

Commit message: Finishing up backup interconnects
Parts:
- removed J3: Conn_01x30, _PanelInterconnct:kyocera_fpc_01x30
- removed SC3, SC4, SC5, SC6, SC7, SC8: Maxeon C60, _PanelInterconnct:maxeon_c60
- J1: footprint _PanelInterconnct:kyocera_fpc_01x10 -> _PanelInterconnects:tb4_10p
- SC1, SC2: footprint _PanelInterconnct:maxeon_c60 -> _PanelInterconnects:maxeon_c60
- moved J1 438.5 mm to (358.4, 148.0), turned to -90 degrees
- moved SC1 333.0 mm to (210.0, 85.0)
- moved SC2 205.5 mm to (210.0, 211.0)
Connections:
- J1 pad 4: unconnected-(J1-Pin_4-Pad4) -> Net-(J1-Pin_1)
- J1 pad 5: Net-(J1-Pin_10) -> Net-(J1-Pin_1)
- SC1 pad 1: Net-(SC1-+) -> Net-(J1-Pin_1)
- SC1 pad 2: Net-(J1-Pin_10) -> Net-(SC1--)
- SC2 pad 1: Net-(SC2-+) -> Net-(J1-Pin_10)
- SC2 pad 2: Net-(SC1-+) -> Net-(SC1--)
Routing:
- net Net-(J1-Pin_1): track 1157.1 -> 0.00 mm, vias 10 -> 0
- net Net-(J1-Pin_10): track 41.0 -> 0.00 mm, vias 21 -> 0
- net Net-(J3-Pin_1): track 30.5 -> 0.00 mm
- added copper zone on B.Cu, net Net-(SC1--)
- added copper zone on F.Cu, net Net-(SC1--)
- removed copper zone on B.Cu, net Net-(J3-Pin_1)
- removed copper zone on F.Cu, net Net-(J3-Pin_1)
- removed copper zone on F.Cu, net Net-(SC1-+)
- removed copper zone on F.Cu, net Net-(SC2-+)
- removed copper zone on F.Cu, net Net-(SC3-+)
- removed copper zone on F.Cu, net Net-(SC4-+)
- removed copper zone on F.Cu, net Net-(SC5-+)
- removed copper zone on F.Cu, net Net-(SC6-+)
- removed copper zone on F.Cu, net Net-(SC7-+)
Other:
- board size 1144.8 x 86.1 mm -> 195.9 x 210.5 mm
- board text removed: "SC2"
- board text removed: "Solar_Cell"

Commit message: Hello
Parts:
- moved J1 36.6 mm to (395.0, 148.0)
Other:
- board size 195.9 x 210.5 mm -> 232.5 x 210.5 mm
Changed lines of the file:
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@@
 	(footprint "_PanelInterconnects:tb4_10p"
 		(layer "F.Cu")
-		(at 358.405 148 -90)
+		(at 395 148 -90)
 		(property "Reference" "J1"
 			(at 0.1 4.33 270)
@@
 	(gr_line
 		(start 274.5 140.35)
-		(end 342.45 140.35)
+		(end 379.04 140.35)
 		(stroke
 			(width 0.05)
@@
 	(gr_line
 		(start 274.5 155.65)
-		(end 342.45 155.65)
+		(end 379.04 155.65)
 		(stroke
 			(width 0.05)
@@
 		(polygon
 			(pts
-				(xy 265 43) (xy 273 43) (xy 273 95.25) (xy 273 142.7) (xy 356.5 142.7) (xy 356.5 147.75) (xy 265 147.75)
+				(xy 265 43) (xy 273 43) (xy 273 95.25) (xy 273 142.7) (xy 393.5 142.7) (xy 393.5 147.75) (xy 265 147.75)
 			)
 		)
@@
 		(polygon
 			(pts
-				(xy 265 148.25) (xy 356.5 148.25) (xy 356.5 153.25) (xy 273 153.25) (xy 273 250.75) (xy 265 250.75)
-			)
-		)
+				(xy 265 148.25) (xy 393.5 148.25) (xy 393.5 153.25) (xy 273 153.25) (xy 273 250.75) (xy 265 250.75)
+			)
+		)

Commit message: Shifitng to single connection
Parts:
- removed J1: Conn_01x10, _PanelInterconnects:tb4_10p
- removed SC1, SC2: Maxeon C60, _PanelInterconnects:maxeon_c60
Routing:
- net Net-(SC1--): vias 0 -> 96
- removed copper zone on B.Cu, net Net-(J1-Pin_1)
- removed copper zone on F.Cu, net Net-(J1-Pin_1)
- removed copper zone on B.Cu, net Net-(J1-Pin_10)
- removed copper zone on F.Cu, net Net-(J1-Pin_10)
Other:
- board size 232.5 x 210.5 mm -> 9 x 210.5 mm
