File: PanelInterconnect.kicad_pcb (KiCad board)
At the start: 2 copper layers, 232.5 x 210.5 mm, 3 parts, among them J1 Conn_01x10

Commit message: Connection to powerboard
Parts:
- removed SC1, SC2: Maxeon C60, _PanelInterconnects:maxeon_c60
- moved J1 54.8 mm to (340.2, 149.2)
Routing:
- net Net-(J1-Pin_10): vias 0 -> 48
- net Net-(J1-Pin_1): vias 0 -> 48
- removed copper zone on B.Cu, net Net-(SC1--)
- removed copper zone on F.Cu, net Net-(SC1--)
Other:
- board size 232.5 x 210.5 mm -> 115.5 x 210.5 mm

Commit message: updated panel interconnect
Parts:
- removed J1: Conn_01x10, _PanelInterconnects:tb4_10p
- added J2: Conn_01x02_Socket, Connector_AMASS:AMASS_XT30U-F_1x02_P5.0mm_Vertical, F.Cu at (301.0, 146.4)
- added SC1: Maxeon C60, _PanelInterconnects:maxeon_c60, F.Cu at (154.5, 86.0)
- added SC2: Maxeon C60, _PanelInterconnects:maxeon_c60, F.Cu at (154.5, 212.0)
Routing:
- net Net-(J2-Pin_2): vias 0 -> 30
- net Net-(J2-Pin_1): vias 0 -> 30
- net Net-(J1-Pin_10): vias 48 -> 0
- net Net-(J1-Pin_1): vias 48 -> 0
- added copper zone on B.Cu, net Net-(J2-Pin_1)
- added copper zone on F.Cu, net Net-(J2-Pin_1)
- added copper zone on B.Cu, net Net-(J2-Pin_2)
- added copper zone on F.Cu, net Net-(J2-Pin_2)
- removed copper zone on B.Cu, net Net-(J1-Pin_1)
- removed copper zone on F.Cu, net Net-(J1-Pin_1)
- removed copper zone on B.Cu, net Net-(J1-Pin_10)
- removed copper zone on F.Cu, net Net-(J1-Pin_10)
Other:
- board size 115.5 x 210.5 mm -> 95 x 212 mm
